Commit message: modifications on launchs and controllrs

File: spot_manipulator_description/urdf/spot.urdf (robot description, URDF)
Before this commit: robot spot, 35 links, 34 joints
Links:
- link Part0_1: mass 6.925827706354272 -> 1
- link Part1_1: mass 12.658281999999998 -> 1
- link Part2_1: mass 7.368455487741179 -> 1
- link Part3_1: mass 10.95245995004642 -> 1
- link Part4_1: mass 3.2278801394086396 -> 1
- link finger_1: mass 1.71236178687828 -> 1
- link gripper_1: mass 5.9780007036604434 -> 1
- link manipulator_base: mass 5.770791545379091 -> 1

File: spot_manipulator_description/urdf/spot_arm.xacro (robot description, xacro)
@@ -7,5 +7,5 @@
   <inertial>
     <origin rpy="0 0 0" xyz="1.2371844231029972e-17 0.0 0.0325"/>
-    <mass value="5.770791545379091"/>
+    <mass value="1"/>
     <inertia ixx="0.007226" ixy="-0.0" ixz="0.0" iyy="0.007226" iyz="0.0" izz="0.010387"/>
   </inertial>
@@ -27,5 +27,5 @@
   <inertial>
     <origin rpy="0 0 0" xyz="-0.00911464892336129 0.12606054498393937 5.551115123125783e-17"/>
-    <mass value="10.95245995004642"/>
+    <mass value="1"/>
     <inertia ixx="0.066789" ixy="0.011971" ixz="-0.0" iyy="0.014993" iyz="0.0" izz="0.071949"/>
   </inertial>
@@ -47,5 +47,5 @@
   <inertial>
     <origin rpy="0 0 0" xyz="-8.366123908053191e-08 0.07051371901138614 0.017123167388316526"/>
-    <mass value="5.9780007036604434"/>
+    <mass value="1"/>
     <inertia ixx="0.01723" ixy="0.0" ixz="0.0" iyy="0.00734" iyz="-0.003871" izz="0.0153"/>
   </inertial>
@@ -67,5 +67,5 @@
   <inertial>
     <origin rpy="0 0 0" xyz="0.8635899028063472 0.09862056591557622 0.00850232975194119"/>
-    <mass value="1.71236178687828"/>
+    <mass value="1"/>
     <inertia ixx="0.002129" ixy="0.0" ixz="-0.0" iyy="0.001681" iyz="0.000162" izz="0.003403"/>
   </inertial>
@@ -87,5 +87,5 @@
   <inertial>
     <origin rpy="0 0 0" xyz="-0.0163095589512068 0.17540914221218962 0.0"/>
-    <mass value="12.658281999999998"/>
+    <mass value="1"/>
     <inertia ixx="0.12979" ixy="0.002625" ixz="0.0" iyy="0.01004" iyz="0.0" izz="0.129493"/>
   </inertial>
@@ -107,5 +107,5 @@
   <inertial>
     <origin rpy="0 0 0" xyz="0.05071972800114364 -1.0308563411658574e-17 0.04676911608650795"/>
-    <mass value="6.925827706354272"/>
+    <mass value="1"/>
     <inertia ixx="0.01241" ixy="-0.0" ixz="-0.001047" iyy="0.010387" iyz="0.0" izz="0.012306"/>
   </inertial>
@@ -127,5 +127,5 @@
   <inertial>
     <origin rpy="0 0 0" xyz="0.03954999709763633 0.03472006124891969 4.209155544249166e-08"/>
-    <mass value="3.2278801394086396"/>
+    <mass value="1"/>
     <inertia ixx="0.00339" ixy="-2.1e-05" ixz="0.0" iyy="0.002242" iyz="-0.0" izz="0.003439"/>
   </inertial>
@@ -147,5 +147,5 @@
   <inertial>
     <origin rpy="0 0 0" xyz="-0.015621881612358529 0.06665620790957599 -0.058074231003688394"/>
-    <mass value="7.368455487741179"/>
+    <mass value="1"/>
     <inertia ixx="0.018073" ixy="0.000915" ixz="-0.00101" iyy="0.011789" iyz="0.003728" izz="0.01667"/>
   </inertial>
