Commit message: adjustments in the inertia matrices to adjust the masses that have been changed.

File: spot_manipulator_description/urdf/spot.urdf.xacro (robot description, xacro)
@@ -23,10 +23,10 @@
     <link name="base_link"/>
     <joint name="base_link_joint" type="fixed">
-        <origin xyz="0 0 0" rpy="0 0 0" />
+        <origin xyz="0 0 0.1" rpy="0 0 0" />
         <parent link="body" />
         <child link="base_link" />
     </joint>
     <joint name="spot_manipulator_joint" type="fixed">
-        <origin xyz="0.3 -0.05 0.09" rpy="0.0 0.0 0.0" />
+        <origin xyz="0 0 0.1" rpy="0.0 0.0 0.0" />
         <parent link="base_link" />
         <child link="manipulator_base" />
@@ -64,8 +64,8 @@
         </plugin>
     </gazebo>
-    <!-- <gazebo>
+    <gazebo>
         <plugin name="gazebo_ros_control" filename="libgazebo_ros_control.so">
             <legacyModeNS>true</legacyModeNS>
         </plugin>
-    </gazebo> -->
+    </gazebo>
 </robot>

File: spot_manipulator_description/urdf/spot_arm.xacro (robot description, xacro)
@@ -3,10 +3,10 @@
 <xacro:include filename="$(find spot_arm_description)/urdf/materials.xacro" />
 <xacro:include filename="$(find spot_manipulator_description)/urdf/spot_arm.trans" />
-<xacro:include filename="$(find spot_arm_description)/urdf/spot_arm.gazebo" />
+<xacro:include filename="$(find spot_manipulator_description)/urdf/spot_arm.gazebo" />
 <link name="manipulator_base">
   <inertial>
     <origin rpy="0 0 0" xyz="1.2371844231029972e-17 0.0 0.0325"/>
-    <mass value="1"/>
-    <inertia ixx="0.007226" ixy="-0.0" ixz="0.0" iyy="0.007226" iyz="0.0" izz="0.010387"/>
+    <mass value="0.1"/>
+    <inertia ixx="0.0001252" ixy="-0.0" ixz="0.0" iyy="0.0001252" iyz="0.0" izz="0.00018"/>
   </inertial>
   <visual>
@@ -27,6 +27,6 @@
   <inertial>
     <origin rpy="0 0 0" xyz="-0.00911464892336129 0.12606054498393937 5.551115123125783e-17"/>
-    <mass value="1"/>
-    <inertia ixx="0.066789" ixy="0.011971" ixz="-0.0" iyy="0.014993" iyz="0.0" izz="0.071949"/>
+    <mass value="0.1"/>
+    <inertia ixx="0.00045" ixy="0.0" ixz="0.0" iyy="0.0004357" iyz="0.0" izz="0.0004369"/>
   </inertial>
   <visual>
@@ -47,6 +47,6 @@
   <inertial>
     <origin rpy="0 0 0" xyz="-8.366123908053191e-08 0.07051371901138614 0.017123167388316526"/>
-    <mass value="1"/>
-    <inertia ixx="0.01723" ixy="0.0" ixz="0.0" iyy="0.00734" iyz="-0.003871" izz="0.0153"/>
+    <mass value="0.1"/>
+    <inertia ixx="0.00026875" ixy="0.0" ixz="-0.0" iyy="0.00025584" iyz="0.0" izz="0.00024338"/>
   </inertial>
   <visual>
@@ -67,19 +67,19 @@
   <inertial>
     <origin rpy="0 0 0" xyz="0.8635899028063472 0.09862056591557622 0.00850232975194119"/>
-    <mass value="1"/>
-    <inertia ixx="0.002129" ixy="0.0" ixz="-0.0" iyy="0.001681" iyz="0.000162" izz="0.003403"/>
-  </inertial>
-  <visual>
+    <mass value="0.1"/>
+    <inertia ixx="0.0002724" ixy="0.0" ixz="-0.0" iyy="0.00224" iyz="0.0" izz="0.0002008"/>
+  </inertial>
+  <visual>
+    <origin rpy="0 0 0" xyz="0.10297709 -0.823505 -0.0185"/>
+    <geometry>
+      <mesh filename="package://spot_arm_description/meshes/finger_1.stl" scale="0.001 0.001 0.001"/>
+    </geometry>
+    <material name="silver"/>
+  </visual>
+  <collision>
     <origin rpy="0 0 0" xyz="0.87709 -0.823505 -0.0185"/>
     <geometry>
       <mesh filename="package://spot_arm_description/meshes/finger_1.stl" scale="0.001 0.001 0.001"/>
     </geometry>
-    <material name="silver"/>
-  </visual>
-  <collision>
-    <origin rpy="0 0 0" xyz="0.87709 -0.823505 -0.0185"/>
-    <geometry>
-      <mesh filename="package://spot_arm_description/meshes/finger_1.stl" scale="0.001 0.001 0.001"/>
-    </geometry>
   </collision>
 </link>
@@ -87,6 +87,6 @@
   <inertial>
     <origin rpy="0 0 0" xyz="-0.0163095589512068 0.17540914221218962 0.0"/>
-    <mass value="1"/>
-    <inertia ixx="0.12979" ixy="0.002625" ixz="0.0" iyy="0.01004" iyz="0.0" izz="0.129493"/>
+    <mass value="0.1"/>
+    <inertia ixx="0.0002724" ixy="0.0" ixz="-0.0" iyy="0.000424" iyz="0.0" izz="0.0001008"/>
   </inertial>
   <visual>
@@ -107,6 +107,6 @@
   <inertial>
     <origin rpy="0 0 0" xyz="0.05071972800114364 -1.0308563411658574e-17 0.04676911608650795"/>
-    <mass value="1"/>
-    <inertia ixx="0.01241" ixy="-0.0" ixz="-0.001047" iyy="0.010387" iyz="0.0" izz="0.012306"/>
+    <mass value="0.1"/>
+    <inertia ixx="0.0002724" ixy="0.0" ixz="-0.0" iyy="0.000224" iyz="0.0" izz="0.0002008"/>
   </inertial>
   <visual>
@@ -127,6 +127,6 @@
   <inertial>
     <origin rpy="0 0 0" xyz="0.03954999709763633 0.03472006124891969 4.209155544249166e-08"/>
-    <mass value="1"/>
-    <inertia ixx="0.00339" ixy="-2.1e-05" ixz="0.0" iyy="0.002242" iyz="-0.0" izz="0.003439"/>
+    <mass value="0.1"/>
+    <inertia ixx="0.0001724" ixy="0.0" ixz="-0.0" iyy="0.000124" iyz="0.0" izz="0.0001008"/>
   </inertial>
   <visual>
@@ -147,6 +147,6 @@
   <inertial>
     <origin rpy="0 0 0" xyz="-0.015621881612358529 0.06665620790957599 -0.058074231003688394"/>
-    <mass value="1"/>
-    <inertia ixx="0.018073" ixy="0.000915" ixz="-0.00101" iyy="0.011789" iyz="0.003728" izz="0.01667"/>
+    <mass value="0.1"/>
+    <inertia ixx="0.0002724" ixy="0.0" ixz="-0.0" iyy="0.000224" iyz="0.0" izz="0.0002008"/>
   </inertial>
   <visual>
@@ -179,5 +179,5 @@
 </joint>
 <joint name="Rev7" type="revolute">
-  <origin rpy="0 0 0" xyz="-0.86859 0.043915 -0.029"/>
+  <origin rpy="0 0 0" xyz="-0.086859 0.043915 -0.029"/>
   <parent link="gripper_1"/>
   <child link="finger_1"/>
@@ -193,5 +193,5 @@
 </joint>
 <joint name="Rev9" type="revolute">
-  <origin rpy="0 0 0" xyz="0.0 0.0 0.065"/>
+  <origin rpy="0 0 1.57" xyz="0.0 0.0 0.065"/>
   <parent link="manipulator_base"/>
   <child link="Part0_1"/>
@@ -207,5 +207,5 @@
 </joint>
 <joint name="Rev11" type="revolute">
-  <origin rpy="0 0 0" xyz="0.002 0.3125 0.0"/>
+  <origin rpy="3.14 0 0" xyz="0.002 0.3125 0.0"/>
   <parent link="Part1_1"/>
   <child link="Part2_1"/>
