Commit message: joystick implementation

File: soft_mobile_manipulator_description/urdf/husky_macro.urdf.xacro (robot description, xacro)
@@ -57,5 +57,5 @@
     <link name="${prefix}base_footprint"/>
     <joint name="body_link" type="fixed">
-      <origin xyz="0 0 0.28" rpy="0 0 0" />
+      <origin xyz="-0.001 0 0.25" rpy="0 0 0" />
       <parent link="${prefix}base_link" />
       <child link="manipulator_link" />
