Commit message: implementation of the joint_trajectory_controller that solved the problem of manipulator oscillation

File: soft_mobile_manipulator_description/urdf/cobra.urdf.xacro (robot description, xacro)
@@ -13,5 +13,5 @@
                 <origin xyz="0 0 0.025" rpy="0 0 0"/>
                 <mass value="0.1" />
-                <inertia ixx="0.00025" ixy="0.0" ixz="0.0" iyy="0.00025" iyz="0.0" izz="0.000125"/>
+                <inertia ixx="0.002" ixy="0.0" ixz="0.0" iyy="0.02" iyz="0.0" izz="0.002"/>
             </inertial>
             <collision>
@@ -32,6 +32,6 @@
             <kp>100.0</kp>
             <kd>1.0</kd>
-            <mu1>1.0</mu1>
-            <mu2>1.0</mu2>
+            <mu1>10.0</mu1>
+            <mu2>10.0</mu2>
             <material>Gazebo/Black</material>
             <self_collide>1</self_collide>
@@ -41,5 +41,5 @@
                 <origin xyz="0 0 0.075" rpy="0 0 0"/>
                 <mass value="0.1" />
-                <inertia ixx="0.00025" ixy="0.0" ixz="0.0" iyy="0.00025" iyz="0.0" izz="0.000125"/>
+                <inertia ixx="0.002" ixy="0.0" ixz="0.0" iyy="0.02" iyz="0.0" izz="0.002"/>
             </inertial>
             <collision>
@@ -72,4 +72,5 @@
             <limit lower="-1.5708" upper="1.5708" effort="100.0" velocity="0.5"/>
             <axis xyz="1 0 0"/>
+            <dynamics damping="10" friction="10"/>
             <disable_collision>true</disable_collision>
     	</joint>
@@ -80,4 +81,5 @@
             <limit lower="-1.5708" upper="1.5708" effort="100.0" velocity="0.5"/>
             <axis xyz="0 1 0"/>
+            <dynamics damping="10" friction="10"/>
             <disable_collision>true</disable_collision>
     	</joint>
@@ -108,5 +110,5 @@
             <origin xyz="0 0 0.075" rpy="0 0 0"/>
             <mass value="0.1" />
-            <inertia ixx="0.00025" ixy="0.0" ixz="0.0" iyy="0.00025" iyz="0.0" izz="0.000125"/>
+            <inertia ixx="0.002" ixy="0.0" ixz="0.0" iyy="0.02" iyz="0.0" izz="0.002"/>
         </inertial>
         <collision>
@@ -126,6 +128,6 @@
         <kp>100000000000000.0</kp>
         <kd>1.0</kd>
-        <mu1>10.0</mu1>
-        <mu2>10.0</mu2>
+        <mu1>1.0</mu1>
+        <mu2>1.0</mu2>
         <material>Gazebo/Green</material>
         <self_collide>0</self_collide>

Commit message: placed an imu in each section to locate

File: soft_mobile_manipulator_description/urdf/cobra.urdf.xacro (robot description, xacro)
@@ -172,5 +172,5 @@
                 <cylinder length="0.03" radius="0.02" />
             </geometry>
-            <material name="blue" />
+            <!-- <material name="blue" /> -->
         </visual>
         <collision>
@@ -181,91 +181,5 @@
             <self_collide>0</self_collide>
         </collision>
-        <!-- <xacro:inertial_box mass="0.1" x="0.12" y="0.15" z="0.15">
-            <origin xyz="0.0 0 0" rpy="0 0 0"/>
-        </xacro:inertial_box> -->
     </link>
-    <!-- <ros2_control name="GazeboSystem" type="system">
-      <hardware>
-        <plugin>gazebo_ros2_control/GazeboSystem</plugin>
-      </hardware>
-      <joint name="cobra_body_1_aux_joint">
-        <command_interface name="position"/>
-        <state_interface name="position"/>
-        <state_interface name="velocity"/>
-        <state_interface name="effort"/>
-      </joint>
-      <joint name="cobra_body_1_joint">
-        <command_interface name="position"/>
-        <state_interface name="position"/>
-        <state_interface name="velocity"/>
-        <state_interface name="effort"/>
-      </joint>
-      <joint name="cobra_body_2_aux_joint">
-        <command_interface name="position"/>
-        <state_interface name="position"/>
-        <state_interface name="velocity"/>
-        <state_interface name="effort"/>
-      </joint>
-      <joint name="cobra_body_2_joint">
-        <command_interface name="position"/>
-        <state_interface name="position"/>
-        <state_interface name="velocity"/>
-        <state_interface name="effort"/>
-      </joint>
-      <joint name="cobra_body_3_aux_joint">
-        <command_interface name="position"/>
-        <state_interface name="position"/>
-        <state_interface name="velocity"/>
-        <state_interface name="effort"/>
-      </joint>
-      <joint name="cobra_body_3_joint">
-        <command_interface name="position"/>
-        <state_interface name="position"/>
-        <state_interface name="velocity"/>
-        <state_interface name="effort"/>
-      </joint>
-      <joint name="cobra_body_4_aux_joint">
-        <command_interface name="position"/>
-        <state_interface name="position"/>
-        <state_interface name="velocity"/>
-        <state_interface name="effort"/>
-      </joint>
-      <joint name="cobra_body_4_joint">
-        <command_interface name="position"/>
-        <state_interface name="position"/>
-        <state_interface name="velocity"/>
-        <state_interface name="effort"/>
-      </joint>
-      <joint name="cobra_body_5_aux_joint">
-        <command_interface name="position"/>
-        <state_interface name="position"/>
-        <state_interface name="velocity"/>
-        <state_interface name="effort"/>
-      </joint>
-      <joint name="cobra_body_5_joint">
-        <command_interface name="position"/>
-        <state_interface name="position"/>
-        <state_interface name="velocity"/>
-        <state_interface name="effort"/>
-      </joint>
-      <joint name="cobra_body_6_aux_joint">
-        <command_interface name="position"/>
-        <state_interface name="position"/>
-        <state_interface name="velocity"/>
-        <state_interface name="effort"/>
-      </joint>
-      <joint name="cobra_body_6_joint">
-        <command_interface name="position"/>
-        <state_interface name="position"/>
-        <state_interface name="velocity"/>
-        <state_interface name="effort"/>
-      </joint>
-    </ros2_control> -->
-    <!-- <gazebo>
-        <plugin filename="libgazebo_ros2_control.so" name="gazebo_ros2_control">
-        <robot_sim_type>gazebo_ros2_control/GazeboSystem</robot_sim_type>
-        <parameters>$(find cobra_control)/config/controllers.yaml</parameters>
-        </plugin>
-    </gazebo> -->
     <joint name="camera_optical_joint" type="fixed">
         <origin xyz="0 0 0" rpy="-1.571 0 -1.571" />
@@ -302,3 +216,41 @@
         </sensor>
     </gazebo>
+    <joint name="imu_joint_manipulator" type="fixed">
+        <origin xyz="0.0 0 0.173" rpy="0 0 0" />
+        <parent link="cobra_body_6" />
+        <child link="imu_link_manipulator" />
+    </joint>
+    <link name="imu_link_manipulator"></link>
+    <gazebo reference="imu_link_manipulator">
+      <sensor name="imu_sensor" type="imu">
+      <plugin filename="libgazebo_ros_imu_sensor.so" name="imu_plugin_1">
+          <ros>
+            <remapping>~/out:=imu/data_raw_1</remapping>
+          </ros>
+          <initial_orientation_as_reference>false</initial_orientation_as_reference>
+        </plugin>
+        <always_on>true</always_on>
+        <update_rate>100</update_rate>
+        <visualize>true</visualize>
+      </sensor>
+    </gazebo>
+    <joint name="imu_joint_manipulator_2" type="fixed">
+       <origin xyz="0.0 0 0.15" rpy="0 0 0" />
+       <parent link="cobra_body_3" />
+       <child link="imu_link_manipulator_2" />
+    </joint>
+    <link name="imu_link_manipulator_2"></link>
+    <gazebo reference="imu_link_manipulator_2">
+      <sensor name="imu_sensor_2" type="imu">
+        <plugin filename="libgazebo_ros_imu_sensor.so" name="imu_plugin_2">
+          <ros>
+            <remapping>~/out:=imu/data_raw_2</remapping>
+          </ros>
+          <initial_orientation_as_reference>false</initial_orientation_as_reference>
+        </plugin>
+        <always_on>true</always_on>
+        <update_rate>100</update_rate>
+        <visualize>true</visualize>
+      </sensor>
+    </gazebo>
 </robot>

Commit message: start of localization using imus

File: soft_mobile_manipulator_description/urdf/cobra.urdf.xacro (robot description, xacro)
@@ -160,4 +160,9 @@
     </joint>
     <link name="camera_link">
+        <inertial>
+            <mass value="0.1" />
+            <origin xyz="0 0 0" rpy="0 0 0"/>
+            <inertia ixx="0.001" ixy="0.0" ixz="0.0" iyy="0.001" iyz="0.0" izz="0.001"/>
+        </inertial>
         <visual>
             <origin xyz="-0.03 0 0" rpy="0 0 0"/>
@@ -236,5 +241,5 @@
     </gazebo>
     <joint name="imu_joint_manipulator_2" type="fixed">
-       <origin xyz="0.0 0 0.15" rpy="0 0 0" />
+       <origin xyz="0.0 0 0.14" rpy="0 0 0" />
        <parent link="cobra_body_3" />
        <child link="imu_link_manipulator_2" />
